File: 010_Hardware/010_uTTA_Eagle/uTTA_V1_Measure.brd (EAGLE design)
At the start: 81.8 x 90.5 mm, 239 parts, among them IC101 AD8676, IC111 LT1167, IC112 LM334M, IC121 LT1167, IC122 LM334M, IC131 LT1167, IC132 LM334M, IC141 LT1167, IC142 LM334M, IC151 AD8676, IC301 MAX6675ISA, IC302 MAX6675ISA, IC303 MAX6675ISA, IC304 MAX6675ISA, IC31 TL072D, IC32 LT1004CLP-2.5, T91 BSS138PS, U1 W25Q512JV, U11 NUCLEO_F103_BOT, X111 BU-SMA-GSPECIAL, X121 BU-SMA-GSPECIAL, X131 BU-SMA-GSPECIAL, X141 BU-SMA-GSPECIAL

Commit message: Minor Cleanup of Design
Parts:
- removed C102, C104, C113, C117, C119, C127, C129, C137, C139, C147, C149, C152, C154, C22, C305, C307, C309, C311: 10u/16V, A_Kondensatoren:C0805
- removed C103, C146, C153, C35, C36: 100n/50V, A_Kondensatoren:C0603
- removed D101, D102: BAT46W, A_Dioden:SOD123
- removed D111, D121, D131, D141: 1N4148, A_Dioden:SOD123
- removed D91, D92: MM3Z3V3T1GR, A_Dioden:SOD323-R
- removed IC101, IC151: AD8676, A_Linear_IC:SO08
- removed IC112, IC122, IC132, IC142: LM334M, A_Linear_IC:SO08
- removed IC31: TL072D, A_Linear_IC:SO08
- removed IC32: LT1004CLP-2.5, A_Linear_Technology:TO92-
- removed JP112, JP122, JP132, JP142, JP31: (no value), Connectors jumper:JP1
- removed R113, R123, R133, R143: 10, A_Resistor:R0805
- removed R114, R124, R134, R144: 100, A_Resistor:S64Y
- removed R35: 10k, A_Resistor:R0603
- removed R36: 2k, A_Resistor:R0603
- removed R91, R92: 4k7, A_Resistor:R0603
- removed R94: 100k, A_Resistor:R0603
- removed TP111, TP112, TP121, TP122, TP131, TP132, TP141, TP142: TPC90H30, A_Testpoint:C90H30
- removed TP201, TP202, TP203, TP204: TP, A_Testpoint:C90
- added 51.2, S51.3, S51.4: SS_ESP101, A_Schalter:SS_ESP101
- added C102.1, C102.2, C102.3, C102.4, C104.1, C104.2, C104.3, C104.4, C152.1, C152.3, C22.1, C22.2, C42, C44, C52.1, C52.2, C52.3, C52.4, C54.1, C54.2, C54.3, C54.4: 1u/25V, A_Kondensatoren:C0603
- added C106.1, C106.2, C106.3, C106.4: 330p, A_Kondensatoren:C0603
- added C151.3, C23.2, C41, C43, C45.1, C45.2, C46, C51.1, C51.2, C51.3, C51.4, C53.1, C53.2, C53.3, C53.4: 100n/50V, A_Kondensatoren:C0603
- added D101.1, D101.2, D101.3, D101.4: SD101, A_Dioden:SOD123
- added D51.1, D51.2, D51.3, D51.4: 1N4148, A_Dioden:SOD123
- added IC151.1, IC151.3: MCP602SN, A_Microchip:SO08
- added IC4: AD5664R, A_Analog_Devices:MSOP10
- added IC41: TL074D, A_Linear_IC:SO14
- added IC42: LT1004CLP-2.5, A_Linear_Technology:TO92-
- added IC51.1, IC51.2, IC51.3, IC51.4: OPA2156ID, A_Linear_IC:SO08
- added L31: FBMMZ2012S, A_Ferrite:FB2012
- added R102.1, R102.2, R102.3, R102.4, R41, R42.1, R42.2, R43.1, R43.2, R52.1, R52.2, R52.3, R52.4, R54.1, R54.2, R54.3, R54.4: 1k, A_Resistor:R0603
- added R151.4: 24k9, A_Resistor:R0603
- added R152.4, R21.2, R44.1, R44.2, R51.1, R51.2, R51.3, R51.4, R53.1, R53.2, R53.3, R53.4: 10k, A_Resistor:R0603
- added R153.4: 330R, A_Resistor:R0603
- added R41.1, R41.2: 1k, A_Resistor:S64Y
- added R45.1, R45.2: 2k, A_Resistor:R0603
- added R46.1, R46.2: 5k6, A_Resistor:R0603
- added R55.1, R55.2, R55.3, R55.4: 22R, A_Resistor:R0805
- added SJ21.1, SJ21.2: (no value), jumper:SJ
- added TP106.1, TP106.2, TP106.3, TP106.4: TPC90H30, A_Testpoint:C90H30
- added TP31, TP32, TP41, TP42, TP43, TP44, TP45.1, TP45.2, TP46.1, TP46.2, TP47.1, TP47.2, TP51.1, TP51.2, TP51.3, TP51.4, TP52.1, TP52.2, TP52.3, TP52.4, TP53.1, TP53.2, TP53.3, TP53.4, TP54.1, TP54.2, TP54.3, TP54.4, TP55.1, TP55.2, TP55.3, TP55.4: TP, A_Testpoint:C90
- added U$10: A4L-LOC_CC_BY_NC_SA, WK_frames:A4_LOC_CC_BY_NC_SA
- added U21.2: W25Q512JV, XMC4500_Relax-V1:SO08W
- C303.1, C303.2, C303.3, C303.4: value 10n/50V -> 100n/50V
- C32: value 10u/16V -> 1u/25V; device A_Kondensatoren:C0805 -> A_Kondensatoren:C0603
- C34: value 10u/16V -> 100n/50V; device A_Kondensatoren:C0805 -> A_Kondensatoren:C0603
- D151, D152: value BAT46W -> MM3Z3V3T1GR; device A_Dioden:SOD123 -> A_Dioden:SOD323-R
- R157: value 24k9 -> 4k7
- R158: value 10k -> 100k
- R159: value 330R -> 4k7
- R31: value 1k -> 10k; device A_Resistor:R0805 -> A_Resistor:R0603
- R32: value 10k -> 1k
- R33: value 10k -> 1k; device A_Resistor:S64Y -> A_Resistor:R0603
- R34: device A_Resistor:R0603 -> A_Resistor:S64Y
- moved R32 230.2 mm to (-198.4, 42.8), turned to 0 degrees
- moved C34 227.0 mm to (-195.3, 40.7), flipped to the top, turned to 0 degrees
- moved R34 225.6 mm to (-202.9, 40.7), turned to 90 degrees
- moved R33 224.9 mm to (-198.4, 40.7)
- moved C33 177.6 mm to (-138.4, 24.9), flipped to the top, turned to 180 degrees
- moved R31 170.9 mm to (-127.6, 23.5)
- moved C31 169.4 mm to (-137.7, 27.9), flipped to the top, turned to 0 degrees
- moved C32 165.3 mm to (-132.0, 29.8), flipped to the top, turned to 0 degrees
- moved D151 27.6 mm to (4.92, 51.8), flipped to the bottom
- moved D152 23.5 mm to (6.67, 51.8), flipped to the bottom, turned to 270 degrees
- moved R158 20.2 mm to (8.57, 51.6), flipped to the bottom, turned to 90 degrees
- moved R157 18.1 mm to (7.46, 55.6), flipped to the bottom, turned to 270 degrees
- moved R159 17.8 mm to (4.13, 55.6), flipped to the bottom, turned to 270 degrees
- renumbered C101 to C151.1, C105 to C153.1, C106 to C153.2, C111 to C105.1, C112 to C107.1, C116 to C101.1, C118 to C103.1, C121 to C105.2, C122 to C107.2, C126 to C101.2, C128 to C103.2, C131 to C105.3, C132 to C107.3, C136 to C101.3, C138 to C103.3, C141 to C105.4, C142 to C107.4, C148 to C103.4, C151 to C101.4, C155 to C153.3, C156 to C153.4, C23 to C23.1, C301 to C301.1, C302 to C301.2, C303 to C301.3, C304 to C301.4, C306 to C303.4, C308 to C303.3, C310 to C303.2, C312 to C303.1, IC111 to IC101.1, IC121 to IC101.2, IC131 to IC101.3, IC141 to IC101.4, IC301 to IC301.1, IC302 to IC301.2, IC303 to IC301.3, IC304 to IC301.4, JP111 to JP101.1, JP121 to JP101.2, JP131 to JP101.3, JP141 to JP101.4, L111 to L101.1, L112 to L102.1, L121 to L101.2, L122 to L102.2, L131 to L101.3, L132 to L102.3, L141 to L101.4, L142 to L102.4, L301 to L301.1, L302 to L302.1, L303 to L301.2, L304 to L302.2, L305 to L301.3, L306 to L302.3, L307 to L301.4, L308 to L302.4, R101 to R151.1, R102 to R154A, R103 to R154B, R104 to R155A, R105 to R156B, R106 to R153.1, R107 to R151.2, R108 to R152.2, R109 to R153.2, R111 to R101.1, R112 to R103.1, R121 to R101.2, R122 to R103.2, R131 to R101.3, R132 to R103.3, R141 to R101.4, R142 to R103.4, R151 to R151.3, R152 to R152.3, R156 to R153.3, R21 to R21.1, R301 to R301.1, R302 to R301.2, R303 to R301.3, R304 to R301.4, R93 to R160, T91 to T151, TP101 to TP151.1, TP102 to TP152.1, TP103 to TP153, TP104 to TP154, TP105 to TP153.1, TP106 to TP151.2, TP107 to TP152.2, TP108 to TP153.2, TP113 to TP101.1, TP114 to TP102.1, TP115 to TP103.1, TP116 to TP104.1, TP117 to TP107.1, TP118 to TP105.1, TP123 to TP101.2, TP124 to TP102.2, TP125 to TP103.2, TP126 to TP104.2, TP127 to TP107.2, TP128 to TP105.2, TP133 to TP101.3, TP135 to TP103.3, TP136 to TP104.3, TP137 to TP107.3, TP138 to TP105.3, TP143 to TP101.4, TP144 to TP102.4, TP145 to TP103.4, TP146 to TP104.4, TP147 to TP107.4, TP148 to TP105.4, TP151 to TP151.3, TP152 to TP152.3, TP155 to TP153.3, TP156 to TP151.4, TP157 to TP152.4, TP158 to TP153.4, TP34 to TP102.3, U1 to U21.1, X111 to X101.1, X121 to X101.2, X131 to X101.3, X141 to X101.4
Connections:
- removed net +8V: C101.3.1, C137.1, IC101.3.7
- removed net AMP1_FB: IC101.2, R151.1.1, R154A.2, R154B.2, R155A.2, R156B.2, TP152.1.P$1
- removed net IS1_R: IC112.1, R113.2
- removed net IS1_RR: R113.1, R114.A
- removed net IS1_TRIM: D111.A, IC112.2, IC112.3, IC112.6, IC112.7, R114.E, R114.S
- removed net IS2_R: IC122.1, R123.2
- removed net IS2_RR: R123.1, R124.A
- removed net IS2_TRIM: D121.A, IC122.2, IC122.3, IC122.6, IC122.7, R124.E, R124.S
- removed net IS3_R: IC132.1, R133.2
- removed net IS3_RR: R133.1, R134.A
- removed net IS3_TRIM: D131.A, IC132.2, IC132.3, IC132.6, IC132.7, R134.E, R134.S
- removed net IS4_R: IC142.1, R143.2
- removed net IS4_RR: R143.1, R144.A
- removed net IS4_TRIM: D141.A, IC142.2, IC142.3, IC142.6, IC142.7, R144.E, R144.S
- removed net I_SEN1: D111.C, JP112.1
- removed net I_SEN2: D121.C, JP122.1
- removed net I_SEN3: D131.C, JP132.1
- removed net I_SEN4: D141.C, JP142.1
- removed net PGA_DIODE1_OUT_AI: C153.1.1, D101.C, R153.1.1, TP153.1.P$1, U11.R_PB11
- removed net VREF_RR: R32.1, R33.A
- removed net V_OFF: IC31.7, R103.1.1, R103.2.1, R103.3.1, R103.4.1, R36.1, TP204.P$1
- new net !DAC_SPI_CSN_DO: IC4.6, R31.2, TP32.P$1
- new net CH1_OFFS: IC4.4, R43.1.1
- new net CH2_4_OFFS: IC4.5, R43.2.1
- new net DIODE2_IN: C106.2.1, C153.1.1, D101.2.C, IC151.1.5, R102.2.1, R153.1.1, TP106.2.P$1, TP153.1.P$1, U11.R_PB11
- new net DIODE3_IN: C106.3.1, D101.3.C, IC151.3.3, R102.3.1, TP106.3.P$1
- new net DIODE4_IN: C106.4.1, D101.4.C, IC151.3.5, R102.4.1, TP106.4.P$1
- new net N$10: D51.1.A, IC51.1.5, R55.1.2, TP55.1.P$1
- new net N$11: IC51.1.1, R54.1.2, R55.1.1, TP54.1.P$1
- new net N$12: IC51.1.3, R51.1.2, R52.1.1, TP51.1.P$1
- new net N$13: IC51.1.2, R53.1.2, R54.1.1, TP52.1.P$1
- new net N$14: IC51.2.3, R51.2.2, R52.2.1, TP51.2.P$1
- new net N$15: IC51.2.2, R53.2.2, R54.2.1, TP52.2.P$1
- new net N$16: IC51.3.6, IC51.3.7, R52.3.2, TP53.3.P$1
- new net N$17: D51.3.A, IC51.3.5, R55.3.2, TP55.3.P$1
- new net N$18: IC51.3.1, R54.3.2, R55.3.1, TP54.3.P$1
- new net N$19: IC51.3.3, R51.3.2, R52.3.1, TP51.3.P$1
- new net N$20: IC51.3.2, R53.3.2, R54.3.1, TP52.3.P$1
- new net N$21: IC51.4.6, IC51.4.7, R52.4.2, TP53.4.P$1
- new net N$22: D51.4.A, IC51.4.5, R55.4.2, TP55.4.P$1
- new net N$23: IC51.4.1, R54.4.2, R55.4.1, TP54.4.P$1
- new net N$24: IC51.4.3, R51.4.2, R52.4.1, TP51.4.P$1
- new net N$25: IC51.4.2, R53.4.2, R54.4.1, TP52.4.P$1
- new net N$26: 51.2.C, R51.2.1
- new net N$27: R51.3.1, S51.3.C
- new net N$28: R51.4.1, S51.4.C
- new net N$29: 51.2.B, IC41.13, IC41.14, R51.1.1, S51.3.B, S51.4.B, TP44.P$1
- new net N$3: C32.1, C33.1, IC4.9, L31.2, TP31.P$1
- new net N$30: IC4.2
- new net N$31: IC4.1, R32.1
- new net N$32: C34.1, IC41.12, R32.2, R33.2, TP43.P$1
- new net N$34: R33.1, R34.S
- new net N$4: IC51.1.6, IC51.1.7, R52.1.2, TP53.1.P$1
- new net N$5: R21.1.2, SJ21.1.2, U21.1.1
- new net N$6: R21.2.2, SJ21.2.2, U21.2.1
- new net N$7: IC51.2.6, IC51.2.7, R52.2.2, TP53.2.P$1
- new net N$8: D51.2.A, IC51.2.5, R55.2.2, TP55.2.P$1
- new net N$9: IC51.2.1, R54.2.2, R55.2.1, TP54.2.P$1
- new net PGA_DIODE1_IN: C106.1.1, D101.1.C, IC151.1.3, R102.1.1, TP106.1.P$1
- new net TP152.1: IC151.1.2, R151.1.1, R154A.2, R154B.2, R155A.2, R156B.2, TP152.1.P$1
- new net VOFFS_RR1: IC41.9, R44.2.1, R45.2.2, TP46.2.P$1
- new net VREF_RR1: R41.1.A, R46.1.1
- new net VREF_RR2: R41.2.A, R46.2.1
- new net VREF_TRIM1: R41.2.S, R42.2.1
- new net V_OFF1: IC41.7, R103.1.1, R45.1.1, TP47.1.P$1
- new net V_OFF2_4: IC41.8, R103.2.1, R103.3.1, R103.4.1, R45.2.1, TP47.2.P$1
- new net V_OFFS_2_4: C45.2.1, IC41.10, R42.2.2, R43.2.2, TP45.2.P$1
- net !SD_SPI_CSN_DO: now also SJ21.1.1, SJ21.2.1; no longer R21.1.2, U21.1.1
- net +15V: no longer C113.1, IC112.4, IC122.4, IC132.4, IC142.4
- net +3V3: now also C151.1.1, C151.3.1, C152.1.1, C152.3.1, C31.1, IC151.1.8, IC151.3.8, L31.1, R31.1; no longer C305.1, C307.1, C309.1, C311.1
- net +5V: now also C101.3.1, C102.1.1, C102.2.1, C102.3.1, C102.4.1, C41.1, C42.1, C51.1.1, C51.2.1, C51.3.1, C51.4.1, C52.1.1, C52.2.1, C52.3.1, C52.4.1, IC101.3.7, IC41.4, IC51.1.8, IC51.2.8, IC51.3.8, IC51.4.8, R41.1; no longer C102.1, C117.1, C127.1, C146.1, C147.1, C151.1.1, C152.1, C31.1, C32.1, IC101.8, IC151.8, IC31.8, R31.2
- net +5V/4: now also C22.1.1, C22.2.1, C23.2.1, R21.2.1, U21.2.3, U21.2.7, U21.2.8; no longer C22.1
- net -5V: now also C104.1.2, C104.2.2, C104.3.2, C104.4.2, C43.2, C44.2, C53.1.2, C53.2.2, C53.3.2, C53.4.2, C54.1.2, C54.2.2, C54.3.2, C54.4.2, IC41.11, IC51.1.4, IC51.2.4, IC51.3.4, IC51.4.4; no longer C103.2, C104.2, C119.2, C129.2, C139.2, C149.2, C153.2, C154.2, C33.2, C34.2, IC101.4, IC151.4, IC31.4
- net AGND: now also 51.2.A, C102.1.2, C102.2.2, C102.3.2, C102.4.2, C104.1.1, C104.2.1, C104.3.1, C104.4.1, C106.1.2, C106.2.2, C106.3.2, C106.4.2, C151.3.2, C152.1.2, C152.3.2, C22.1.2, C22.2.2, C23.2.2, C33.2, C34.2, C41.2, C42.2, C43.1, C44.1, C45.1.2, C45.2.2, C46.2, C51.1.2, C51.2.2, C51.3.2, C51.4.2, C52.1.2, C52.2.2, C52.3.2, C52.4.2, C53.1.1, C53.2.1, C53.3.1, C53.4.1, C54.1.1, C54.2.1, C54.3.1, C54.4.1, D101.1.A, D101.2.A, D101.3.A, D101.4.A, IC151.1.4, IC151.3.4, IC4.3, IC42.1, R152.4.1, R34.E, R41.1.E, R41.2.E, R53.1.1, R53.2.1, R53.3.1, R53.4.1, S51.3.A, S51.4.A, U21.2.4; no longer C102.2, C103.1, C104.1, C113.2, C117.2, C119.1, C127.2, C129.1, C137.2, C139.1, C146.2, C147.2, C149.1, C152.2, C153.1, C154.1, C22.2, C305.2, C307.2, C309.2, C311.2, C33.1, C34.1, C35.2, C36.2, D101.A, D102.A, D91.A, D92.A, IC32.1, JP31.2, R33.E, R94.1
- net AMP1_OUT: now also IC151.1.1; no longer IC101.1
- net AMP2_FB: now also IC151.1.6; no longer IC101.6
- net AMP2_OUT: now also IC151.1.7; no longer IC101.7
- net AMP3_FB: now also IC151.3.2; no longer IC151.2
- net AMP3_OUT: now also IC151.3.1; no longer IC151.1
- net AMP4_FB: now also IC151.3.6, R151.4.1, R152.4.2; no longer IC151.6, R157.1, R158.2
- net AMP4_OUT: now also IC151.3.7, R151.4.2, R153.4.2; no longer IC151.7, R157.2, R159.2
- net B0_GATE: now also D151.C, R159.2; no longer D92.C, R92.2
- net B1_GATE: now also D152.C, R157.2, R158.2; no longer D91.C, R91.2, R94.2
- net DIFF_AMP1_OUT: now also R102.1.2; no longer IC101.3
- net DIFF_AMP2_OUT: now also R102.2.2; no longer IC101.5
- net DIFF_AMP3_OUT: now also R102.3.2; no longer IC151.3
- net DIFF_AMP4_OUT: now also R102.4.2; no longer IC151.5
- net DIODE2_OUT_AI: no longer D102.C
- net DIODE3_OUT_AI: no longer D151.C
- net DIODE4_OUT_AI: now also R153.4.1; no longer D152.C, R159.1
- net GAIN_B0_DO: now also R159.1; no longer R92.1
- net GAIN_B1_DO: now also R157.1; no longer R91.1
- net SD_SPI_MISO_DI: now also U21.2.2
- net SD_SPI_MOSI_DO: now also IC4.8, U21.2.5
- net SD_SPI_SCK_DO: now also IC4.7, U21.2.6
- net SENSE1+: now also D51.1.C; no longer JP112.2, TP112.P$1
- net SENSE1-: no longer TP111.P$1
- net SENSE2+: now also D51.2.C; no longer JP122.2, TP122.P$1
- net SENSE2-: no longer TP121.P$1
- net SENSE3+: now also D51.3.C; no longer JP132.2, TP132.P$1
- net SENSE3-: no longer TP131.P$1
- net SENSE4+: now also D51.4.C; no longer JP142.2, TP142.P$1
- net SENSE4-: no longer TP141.P$1
- net VOFFS_RR: now also IC41.6, R44.1.1, R45.1.2, TP46.1.P$1; no longer IC31.6, R35.1, R36.2, TP203.P$1
- net VREF: now also C46.1, IC41.3, IC42.2, R41.2, TP41.P$1; no longer C35.1, IC31.3, IC32.2, R31.1
- net VREF_2V5_BUFF: now also IC4.10, IC41.1, IC41.2, R34.A, R44.1.2, R44.2.2, R46.1.2, R46.2.2, TP42.P$1; no longer IC31.1, IC31.2, R32.2, R35.2, TP201.P$1
- net VREF_TRIM: now also R41.1.S, R42.1.1; no longer R33.S, R34.1
- net V_OFFS: now also C45.1.1, IC41.5, R42.1.2, R43.1.2, TP45.1.P$1; no longer C36.1, IC31.5, JP31.1, R34.2, TP202.P$1
Routing:
- net V_OFF: track 85.2 -> 0.00 mm, vias 5 -> 0
- net V_OFF1: track 0.00 -> 68.8 mm, vias 0 -> 5
- net PGA_DIODE1_OUT_AI: track 34.5 -> 0.00 mm, vias 1 -> 0
- net DIODE2_IN: track 0.00 -> 34.2 mm, vias 0 -> 1
- net IS4_TRIM: track 25.4 -> 0.00 mm
- net IS1_TRIM: track 25.4 -> 0.00 mm
- net IS3_TRIM: track 25.4 -> 0.00 mm
- net IS2_TRIM: track 25.3 -> 0.00 mm
- net -5V: track 39.3 -> 15.4 mm, vias 7 -> 4
- net +3V3: track 81.4 -> 59.2 mm
- net +5V: track 32.3 -> 16.0 mm, vias 7 -> 5
- net AGND: track 20.8 -> 5.50 mm, vias 25 -> 20
- net VREF_2V5_BUFF: track 11.9 -> 0.00 mm
- net TP152.1: track 0.00 -> 11.8 mm
- net AMP1_FB: track 11.7 -> 0.00 mm
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