File: 010_Hardware/010_uTTA_Eagle/uTTA_V1_Measure.sch (EAGLE design)
At the start: 238 parts, among them IC101 AD8676, IC111 LT1167, IC112 LM334M, IC121 LT1167, IC122 LM334M, IC131 LT1167, IC132 LM334M, IC141 LT1167, IC142 LM334M, IC151 AD8676, IC301 MAX6675ISA, IC302 MAX6675ISA, IC303 MAX6675ISA, IC304 MAX6675ISA, IC31 TL072D, IC32 LT1004CLP-2.5, T91 BSS138PS, U1 W25Q512JV, U11 NUCLEO_F103_BOT, X111 BU-SMA-GSPECIAL, X121 BU-SMA-GSPECIAL, X131 BU-SMA-GSPECIAL, X141 BU-SMA-GSPECIAL

Commit message: Minor Cleanup of Design
Parts:
- removed C101, C103, C112, C116, C118, C122, C126, C128, C151, C153, C35, C36: 100n/50V, A_Kondensatoren:C-EUC0603
- removed C102, C104, C113, C117, C119, C127, C129, C137, C139, C147, C149, C152, C154, C22, C305, C307, C309, C311: 10u/16V, A_Kondensatoren:C-EUC0805
- removed C105, C106, C155: 1n/25V, A_Kondensatoren:C-EUC0603
- removed C111, C121: 10p, A_Kondensatoren:C-EUC0603
- removed C301, C302, C303, C304, C306, C308, C310, C312: 10n/50V, A_Kondensatoren:C-EUC0603
- removed D101, D102: BAT46W, A_Dioden:DIODE-SOD123
- removed D111, D121, D131, D141: 1N4148, A_Dioden:DIODE-SOD123
- removed D91, D92: MM3Z3V3T1GR, A_Dioden:MM3Z3V3T1GR
- removed IC101, IC151: AD8676, A_Linear_IC:OPA2192
- removed IC111, IC121: LT1167, A_Linear_Technology:LT1167
- removed IC112, IC122, IC132, IC142: LM334M, A_Linear_IC:LM334M
- removed IC301, IC302, IC303, IC304: MAX6675ISA, A_MAXIM_IC:MAX6675ISA
- removed IC31: TL072D, A_Linear_IC:TL072D
- removed IC32: LT1004CLP-2.5, A_Linear_Technology:LT1004CLP-2.5
- removed JP111, JP112, JP121, JP122, JP132, JP142, JP31: (no value), Connectors jumper:JP1E
- removed L111, L112, L121, L122, L301, L302, L303, L304, L305, L306, L307, L308: FBMMZ2012S, A_Ferrite:FBMMZ2012S
- removed R101, R107, R151: 24k9, A_Resistor:R-EU_R0603
- removed R102, R103, R93, R94: 100k, A_Resistor:R-EU_R0603
- removed R104: 15K, A_Resistor:R-EU_R0603
- removed R105: DNP, A_Resistor:R-EU_R0603
- removed R106, R109, R156: 330R, A_Resistor:R-EU_R0603
- removed R108, R152, R21, R301, R302, R303, R304, R35: 10k, A_Resistor:R-EU_R0603
- removed R111, R121: 49k4, A_Resistor:R-EU_R0805
- removed R112, R122: 10R, A_Resistor:R-EU_R0603
- removed R113, R123, R133, R143: 10, A_Resistor:R-EU_R0805
- removed R114, R124, R134, R144: 100, A_Resistor:TRIM_EU-S64Y
- removed R36: 2k, A_Resistor:R-EU_R0603
- removed R91, R92: 4k7, A_Resistor:R-EU_R0603
- removed T91: BSS138PS, A_Transistoren:BSS138PS
- removed TP101, TP102, TP103, TP104, TP106, TP107, TP113, TP114, TP115, TP116, TP117, TP118, TP123, TP124, TP125, TP126, TP127, TP128, TP151, TP201, TP202, TP203, TP204: TP, A_Testpoint:TP
- removed TP105, TP108, TP111, TP112, TP121, TP122, TP131, TP132, TP141, TP142, TP152, TP155, TP156, TP157: TPC90H30, A_Testpoint:TPC90H30
- removed U1: W25Q512JV, XMC4500_Relax-V1:W25Q80BVSSIG
- removed X111, X121: BU-SMA-GSPECIAL, A_Steckverbinder:BU-SMA-GSPECIAL
- added 51.2, S51.3, S51.4: SS_ESP101, A_Schalter:SS_ESP101
- added C101.3, C101.4, C103.3, C103.4, C107.3, C107.4, C151.1, C151.3, C23.2, C303.1, C303.2, C303.3, C303.4, C41, C43, C45.1, C45.2, C46, C51.1, C51.2, C51.3, C51.4, C53.1, C53.2, C53.3, C53.4: 100n/50V, A_Kondensatoren:C-EUC0603
- added C102.1, C102.2, C102.3, C102.4, C104.1, C104.2, C104.3, C104.4, C152.1, C152.3, C22.1, C22.2, C42, C44, C52.1, C52.2, C52.3, C52.4, C54.1, C54.2, C54.3, C54.4: 1u/25V, A_Kondensatoren:C-EUC0603
- added C105.3, C105.4: 10p, A_Kondensatoren:C-EUC0603
- added C106.1, C106.2, C106.3, C106.4: 330p, A_Kondensatoren:C-EUC0603
- added C153.1, C153.3, C153.4: 1n/25V, A_Kondensatoren:C-EUC0603
- added C301.1, C301.2, C301.3, C301.4: 10n/50V, A_Kondensatoren:C-EUC0603
- added D101.1, D101.2, D101.3, D101.4: SD101, A_Dioden:DIODE-SOD123
- added D51.1, D51.2, D51.3, D51.4: 1N4148, A_Dioden:DIODE-SOD123
- added IC101.3, IC101.4: LT1167, A_Linear_Technology:LT1167
- added IC151.1, IC151.3: MCP602SN, A_Microchip:MCP602SN
- added IC301.1, IC301.2, IC301.3, IC301.4: MAX6675ISA, A_MAXIM_IC:MAX6675ISA
- added IC4: AD5664R, A_Analog_Devices:AD5664R
- added IC41: TL074D, A_Linear_IC:TL074D
- added IC42: LT1004CLP-2.5, A_Linear_Technology:LT1004CLP-2.5
- added IC51.1, IC51.2, IC51.3, IC51.4: OPA2156ID, A_Linear_IC:OPA2156ID
- added JP101.3, JP101.4: (no value), Connectors jumper:JP1E
- added L101.3, L101.4, L102.3, L102.4, L301.1, L301.2, L301.3, L301.4, L302.1, L302.2, L302.3, L302.4, L31: FBMMZ2012S, A_Ferrite:FBMMZ2012S
- added R101.3, R101.4: 49k4, A_Resistor:R-EU_R0805
- added R102.1, R102.2, R102.3, R102.4, R41, R42.1, R42.2, R43.1, R43.2, R52.1, R52.2, R52.3, R52.4, R54.1, R54.2, R54.3, R54.4: 1k, A_Resistor:R-EU_R0603
- added R103.3, R103.4: 10R, A_Resistor:R-EU_R0603
- added R151.1, R151.2, R151.3, R151.4: 24k9, A_Resistor:R-EU_R0603
- added R152.2, R152.3, R152.4, R21.1, R21.2, R301.1, R301.2, R301.3, R301.4, R44.1, R44.2, R51.1, R51.2, R51.3, R51.4, R53.1, R53.2, R53.3, R53.4: 10k, A_Resistor:R-EU_R0603
- added R153.1, R153.2, R153.3, R153.4: 330R, A_Resistor:R-EU_R0603
- added R154A, R154B, R160: 100k, A_Resistor:R-EU_R0603
- added R155A: 15K, A_Resistor:R-EU_R0603
- added R156B: DNP, A_Resistor:R-EU_R0603
- added R41.1, R41.2: 1k, A_Resistor:TRIM_EU-S64Y
- added R45.1, R45.2: 2k, A_Resistor:R-EU_R0603
- added R46.1, R46.2: 5k6, A_Resistor:R-EU_R0603
- added R55.1, R55.2, R55.3, R55.4: 22R, A_Resistor:R-EU_R0805
- added SJ21.1, SJ21.2: (no value), jumper:SJ
- added T151: BSS138PS, A_Transistoren:BSS138PS
- added TP101.3, TP101.4, TP102.3, TP102.4, TP103.3, TP103.4, TP104.3, TP104.4, TP105.3, TP105.4, TP107.3, TP107.4, TP151.1, TP151.2, TP151.3, TP152.1, TP152.2, TP153, TP154, TP31, TP32, TP41, TP42, TP43, TP44, TP45.1, TP45.2, TP46.1, TP46.2, TP47.1, TP47.2, TP51.1, TP51.2, TP51.3, TP51.4, TP52.1, TP52.2, TP52.3, TP52.4, TP53.1, TP53.2, TP53.3, TP53.4, TP54.1, TP54.2, TP54.3, TP54.4, TP55.1, TP55.2, TP55.3, TP55.4: TP, A_Testpoint:TP
- added TP106.1, TP106.2, TP106.3, TP106.4, TP151.4, TP152.3, TP152.4, TP153.1, TP153.3, TP153.4: TPC90H30, A_Testpoint:TPC90H30
- added U$10: A4L-LOC_CC_BY_NC_SA, WK_frames:A4L-LOC_CC_BY_NC_SA
- added U21.1, U21.2: W25Q512JV, XMC4500_Relax-V1:W25Q80BVSSIG
- added X101.3, X101.4: BU-SMA-GSPECIAL, A_Steckverbinder:BU-SMA-GSPECIAL
- C31, C33: PACKAGE (none) -> C0603
- C32: value 10u/16V -> 1u/25V; device A_Kondensatoren:C-EUC0805 -> A_Kondensatoren:C-EUC0603; PACKAGE (none) -> C0603
- C34: value 10u/16V -> 100n/50V; device A_Kondensatoren:C-EUC0805 -> A_Kondensatoren:C-EUC0603; PACKAGE (none) -> C0603
- D151, D152: value BAT46W -> MM3Z3V3T1GR; device A_Dioden:DIODE-SOD123 -> A_Dioden:MM3Z3V3T1GR; PACKAGE (none) -> SOD323
- R157: value 24k9 -> 4k7; PACKAGE (none) -> R0603
- R158: value 10k -> 100k
- R159: value 330R -> 4k7; PACKAGE (none) -> R0603
- R31: value 1k -> 10k; device A_Resistor:R-EU_R0805 -> A_Resistor:R-EU_R0603; PACKAGE (none) -> R0603
- R32: value 10k -> 1k; PACKAGE (none) -> R0603
- R33: value 10k -> 1k; device A_Resistor:TRIM_EU-S64Y -> A_Resistor:R-EU_R0603; PACKAGE (none) -> R0603
- R34: device A_Resistor:R-EU_R0603 -> A_Resistor:TRIM_EU-S64Y; PACKAGE (none) -> S64Y
- renumbered C131 to C105.1, C132 to C107.1, C136 to C101.1, C138 to C103.1, C141 to C105.2, C142 to C107.2, C146 to C101.2, C148 to C103.2, C156 to C153.2, C23 to C23.1, IC131 to IC101.1, IC141 to IC101.2, JP131 to JP101.1, JP141 to JP101.2, L131 to L101.1, L132 to L102.1, L141 to L101.2, L142 to L102.2, R131 to R101.1, R132 to R103.1, R141 to R101.2, R142 to R103.2, TP133 to TP101.1, TP135 to TP103.1, TP136 to TP104.1, TP137 to TP107.1, TP138 to TP105.1, TP143 to TP101.2, TP144 to TP102.2, TP145 to TP103.2, TP146 to TP104.2, TP147 to TP107.2, TP148 to TP105.2, TP158 to TP153.2, TP34 to TP102.1, X131 to X101.1, X141 to X101.2
Connections:
- removed net +8V: C101.1.1, C137.1, IC101.1PWR.V+
- removed net AMP1_FB: IC101A.-IN, R101.1, R102.2, R103.2, R104.2, R105.2, TP102.TP
- removed net IS1_R: IC112.R, R113.2
- removed net IS1_RR: R113.1, R114.A
- removed net IS1_TRIM: D111.A, IC112.V-, IC112.V-@1, IC112.V-@2, IC112.V-@3, R114.E, R114.S
- removed net IS2_R: IC122.R, R123.2
- removed net IS2_RR: R123.1, R124.A
- removed net IS2_TRIM: D121.A, IC122.V-, IC122.V-@1, IC122.V-@2, IC122.V-@3, R124.E, R124.S
- removed net IS3_R: IC132.R, R133.2
- removed net IS3_RR: R133.1, R134.A
- removed net IS3_TRIM: D131.A, IC132.V-, IC132.V-@1, IC132.V-@2, IC132.V-@3, R134.E, R134.S
- removed net IS4_R: IC142.R, R143.2
- removed net IS4_RR: R143.1, R144.A
- removed net IS4_TRIM: D141.A, IC142.V-, IC142.V-@1, IC142.V-@2, IC142.V-@3, R144.E, R144.S
- removed net I_SEN1: D111.C, JP112.1
- removed net I_SEN2: D121.C, JP122.1
- removed net I_SEN3: D131.C, JP132.1
- removed net I_SEN4: D141.C, JP142.1
- removed net PGA_DIODE1_OUT_AI: C105.1, D101.C, R106.1, TP105.TP, U11B.PB11
- removed net VREF_RR: R32.1, R33.A
- removed net V_OFF: IC31B.OUT, R103.1.1, R103.2.1, R112.1, R122.1, R36.1, TP204.TP
- new net !DAC_SPI_CSN_DO: IC4.!SYNC, R31.2, TP32.TP
- new net CH1_OFFS: IC4.VOUT_C, R43.1.1
- new net CH2_4_OFFS: IC4.VOUT_D, R43.2.1
- new net DIODE2_IN: C106.2.1, C153.1.1, D101.2.C, IC151.1B.+IN, R102.2.1, R153.1.1, TP106.2.TP, TP153.1.TP, U11B.PB11
- new net DIODE3_IN: C106.3.1, D101.3.C, IC151.3A.+IN, R102.3.1, TP106.3.TP
- new net DIODE4_IN: C106.4.1, D101.4.C, IC151.3B.+IN, R102.4.1, TP106.4.TP
- new net N$10: D51.1.A, IC51.1B.+IN, R55.1.2, TP55.1.TP
- new net N$11: IC51.1A.OUT, R54.1.2, R55.1.1, TP54.1.TP
- new net N$12: IC51.1A.+IN, R51.1.2, R52.1.1, TP51.1.TP
- new net N$13: IC51.1A.-IN, R53.1.2, R54.1.1, TP52.1.TP
- new net N$14: IC51.2A.+IN, R51.2.2, R52.2.1, TP51.2.TP
- new net N$15: IC51.2A.-IN, R53.2.2, R54.2.1, TP52.2.TP
- new net N$16: IC51.3B.-IN, IC51.3B.OUT, R52.3.2, TP53.3.TP
- new net N$17: D51.3.A, IC51.3B.+IN, R55.3.2, TP55.3.TP
- new net N$18: IC51.3A.OUT, R54.3.2, R55.3.1, TP54.3.TP
- new net N$19: IC51.3A.+IN, R51.3.2, R52.3.1, TP51.3.TP
- new net N$20: IC51.3A.-IN, R53.3.2, R54.3.1, TP52.3.TP
- new net N$21: IC51.4B.-IN, IC51.4B.OUT, R52.4.2, TP53.4.TP
- new net N$22: D51.4.A, IC51.4B.+IN, R55.4.2, TP55.4.TP
- new net N$23: IC51.4A.OUT, R54.4.2, R55.4.1, TP54.4.TP
- new net N$24: IC51.4A.+IN, R51.4.2, R52.4.1, TP51.4.TP
- new net N$25: IC51.4A.-IN, R53.4.2, R54.4.1, TP52.4.TP
- new net N$26: 51.2.P, R51.2.1
- new net N$27: R51.3.1, S51.3.P
- new net N$28: R51.4.1, S51.4.P
- new net N$29: 51.2.O, IC41D.-IN, IC41D.OUT, R51.1.1, S51.3.O, S51.4.O, TP44.TP
- new net N$3: C32.1, C33.1, IC4.VDD, L31.2, TP31.TP
- new net N$30: IC4.VOUT_B
- new net N$31: IC4.VOUT_A, R32.1
- new net N$32: C34.1, IC41D.+IN, R32.2, R33.2, TP43.TP
- new net N$34: R33.1, R34.S
- new net N$4: IC51.1B.-IN, IC51.1B.OUT, R52.1.2, TP53.1.TP
- new net N$5: R21.1.2, SJ21.1.2, U21.1.CS#
- new net N$6: R21.2.2, SJ21.2.2, U21.2.CS#
- new net N$7: IC51.2B.-IN, IC51.2B.OUT, R52.2.2, TP53.2.TP
- new net N$8: D51.2.A, IC51.2B.+IN, R55.2.2, TP55.2.TP
- new net N$9: IC51.2A.OUT, R54.2.2, R55.2.1, TP54.2.TP
- new net PGA_DIODE1_IN: C106.1.1, D101.1.C, IC151.1A.+IN, R102.1.1, TP106.1.TP
- new net TP152.1: IC151.1A.-IN, R151.1.1, R154A.2, R154B.2, R155A.2, R156B.2, TP152.1.TP
- new net VOFFS_RR1: IC41C.-IN, R44.2.1, R45.2.2, TP46.2.TP
- new net VREF_RR1: R41.1.A, R46.1.1
- new net VREF_RR2: R41.2.A, R46.2.1
- new net VREF_TRIM1: R41.2.S, R42.2.1
- new net V_OFF1: IC41B.OUT, R103.1.1, R45.1.1, TP47.1.TP
- new net V_OFF2_4: IC41C.OUT, R103.2.1, R103.3.1, R103.4.1, R45.2.1, TP47.2.TP
- new net V_OFFS_2_4: C45.2.1, IC41C.+IN, R42.2.2, R43.2.2, TP45.2.TP
- net !SD_SPI_CSN_DO: now also SJ21.1.1, SJ21.2.1; no longer R21.2, U1.CS#
- net !TEMP_SPI_CSN0_DO: now also IC301.1A.!CSN, R301.1.2; no longer IC301A.!CSN, R301.2
- net !TEMP_SPI_CSN1_DO: now also IC301.2A.!CSN, R301.2.2; no longer IC302A.!CSN, R302.2
- net !TEMP_SPI_CSN2_DO: now also IC301.3A.!CSN, R301.3.2; no longer IC303A.!CSN, R303.2
- net !TEMP_SPI_CSN3_DO: now also IC301.4A.!CSN, R301.4.2; no longer IC304A.!CSN, R304.2
- net +15V: no longer C113.1, IC112.V+, IC122.V+, IC132.V+, IC142.V+
- net +3V3: now also C151.1.1, C151.3.1, C152.1.1, C152.3.1, C303.1.1, C303.2.1, C303.3.1, C303.4.1, C31.1, IC151.1P.V+, IC151.3P.V+, IC301.1P.VCC, IC301.2P.VCC, IC301.3P.VCC, IC301.4P.VCC, L31.1, R301.1.1, R301.2.1, R301.3.1, R301.4.1, R31.1; no longer C305.1, C306.1, C307.1, C308.1, C309.1, C310.1, C311.1, C312.1, IC301P.VCC, IC302P.VCC, IC303P.VCC, IC304P.VCC, R301.1, R302.1, R303.1, R304.1
- net +5V: now also C101.1.1, C101.3.1, C101.4.1, C102.1.1, C102.2.1, C102.3.1, C102.4.1, C41.1, C42.1, C51.1.1, C51.2.1, C51.3.1, C51.4.1, C52.1.1, C52.2.1, C52.3.1, C52.4.1, IC101.1PWR.V+, IC101.3PWR.V+, IC101.4PWR.V+, IC41P.V+, IC51.1PWR.V+, IC51.2PWR.V+, IC51.3PWR.V+, IC51.4PWR.V+, R41.1; no longer C101.1, C102.1, C116.1, C117.1, C126.1, C127.1, C147.1, C151.1, C152.1, C31.1, C32.1, IC101PWR.V+, IC111PWR.V+, IC121PWR.V+, IC151PWR.V+, IC31P.V+, R31.2
- net +5V/4: now also C22.1.1, C22.2.1, C23.2.1, R21.1.1, R21.2.1, U21.1.HOLD#, U21.1.VCC, U21.1.WP#, U21.2.HOLD#, U21.2.VCC, U21.2.WP#; no longer C22.1, R21.1, U1.HOLD#, U1.VCC, U1.WP#
- net -5V: now also C103.3.2, C103.4.2, C104.1.2, C104.2.2, C104.3.2, C104.4.2, C43.2, C44.2, C53.1.2, C53.2.2, C53.3.2, C53.4.2, C54.1.2, C54.2.2, C54.3.2, C54.4.2, IC101.3PWR.V-, IC101.4PWR.V-, IC41P.V-, IC51.1PWR.V-, IC51.2PWR.V-, IC51.3PWR.V-, IC51.4PWR.V-; no longer C103.2, C104.2, C118.2, C119.2, C128.2, C129.2, C139.2, C149.2, C153.2, C154.2, C33.2, C34.2, IC101PWR.V-, IC111PWR.V-, IC121PWR.V-, IC151PWR.V-, IC31P.V-
- net AGND: now also 51.2.S, C101.3.2, C101.4.2, C102.1.2, C102.2.2, C102.3.2, C102.4.2, C103.3.1, C103.4.1, C104.1.1, C104.2.1, C104.3.1, C104.4.1, C106.1.2, C106.2.2, C106.3.2, C106.4.2, C107.3.2, C107.4.2, C151.1.2, C151.3.2, C152.1.2, C152.3.2, C153.1.2, C153.3.2, C153.4.2, C22.1.2, C22.2.2, C23.2.2, C303.1.2, C303.2.2, C303.3.2, C303.4.2, C33.2, C34.2, C41.2, C42.2, C43.1, C44.1, C45.1.2, C45.2.2, C46.2, C51.1.2, C51.2.2, C51.3.2, C51.4.2, C52.1.2, C52.2.2, C52.3.2, C52.4.2, C53.1.1, C53.2.1, C53.3.1, C53.4.1, C54.1.1, C54.2.1, C54.3.1, C54.4.1, D101.1.A, D101.2.A, D101.3.A, D101.4.A, IC151.1P.V-, IC151.3P.V-, IC301.1P.GND, IC301.2P.GND, IC301.3P.GND, IC301.4P.GND, IC4.GND, IC42.A, R152.2.1, R152.3.1, R152.4.1, R160.1, R34.E, R41.1.E, R41.2.E, R53.1.1, R53.2.1, R53.3.1, R53.4.1, S51.3.S, S51.4.S, T151A.S, T151B.S, U21.1.GND, U21.2.GND; no longer C101.2, C102.2, C103.1, C104.1, C105.2, C106.2, C112.2, C113.2, C116.2, C117.2, C118.1, C119.1, C122.2, C126.2, C127.2, C128.1, C129.1, C137.2, C139.1, C147.2, C149.1, C151.2, C152.2, C153.1, C154.1, C155.2, C22.2, C305.2, C306.2, C307.2, C308.2, C309.2, C310.2, C311.2, C312.2, C33.1, C34.1, C35.2, C36.2, D101.A, D102.A, D91.A, D92.A, IC301P.GND, IC302P.GND, IC303P.GND, IC304P.GND, IC32.A, JP31.2, R108.1, R152.1, R33.E, R93.1, R94.1, T91A.S, T91B.S, U1.GND
- net AMP1_OUT: now also IC151.1A.OUT, R151.1.2, R153.1.2, TP151.1.TP; no longer IC101A.OUT, R101.2, R106.2, TP101.TP
- net AMP1_RG_B0: now also R155A.1, R156B.1, T151B.D, TP154.TP; no longer R104.1, R105.1, T91B.D, TP104.TP
- net AMP1_RG_B1: now also R154A.1, R154B.1, T151A.D, TP153.TP; no longer R102.1, R103.1, T91A.D, TP103.TP
- net AMP2_FB: now also IC151.1B.-IN, R151.2.1, R152.2.2, TP152.2.TP; no longer IC101B.-IN, R107.1, R108.2, TP107.TP
- net AMP2_OUT: now also IC151.1B.OUT, R151.2.2, R153.2.2, TP151.2.TP; no longer IC101B.OUT, R107.2, R109.2, TP106.TP
- net AMP3_FB: now also IC151.3A.-IN, R151.3.1, R152.3.2, TP152.3.TP; no longer IC151A.-IN, R151.1, R152.2, TP152.TP
- net AMP3_OUT: now also IC151.3A.OUT, R151.3.2, R153.3.2, TP151.3.TP; no longer IC151A.OUT, R151.2, R156.2, TP151.TP
- net AMP4_FB: now also IC151.3B.-IN, R151.4.1, R152.4.2, TP152.4.TP; no longer IC151B.-IN, R157.1, R158.2, TP157.TP
- net AMP4_OUT: now also IC151.3B.OUT, R151.4.2, R153.4.2, TP151.4.TP; no longer IC151B.OUT, R157.2, R159.2, TP156.TP
- net B0_GATE: now also D151.C, R159.2, R160.2, T151B.G; no longer D92.C, R92.2, R93.2, T91B.G
- net B1_GATE: now also D152.C, R157.2, R158.2, T151A.G; no longer D91.C, R91.2, R94.2, T91A.G
- net DIFF_AMP1_OUT: now also IC101.1A.OUT, R102.1.2, TP105.1.TP; no longer IC101A.+IN, IC111A.OUT, TP118.TP
- net DIFF_AMP2_OUT: now also IC101.2A.OUT, R102.2.2, TP105.2.TP; no longer IC101B.+IN, IC121A.OUT, TP128.TP
- net DIFF_AMP3_OUT: now also IC101.3A.OUT, R102.3.2, TP105.3.TP; no longer IC101.1A.OUT, IC151A.+IN, TP105.1.TP
- net DIFF_AMP4_OUT: now also IC101.4A.OUT, R102.4.2, TP105.4.TP; no longer IC101.2A.OUT, IC151B.+IN, TP105.2.TP
- net DIODE2_OUT_AI: now also C153.2.1, R153.2.1, TP153.2.TP; no longer C106.1, D102.C, R109.1, TP108.TP
- net DIODE3_OUT_AI: now also C153.3.1, R153.3.1, TP153.3.TP; no longer C155.1, D151.C, R156.1, TP155.TP
- net DIODE4_OUT_AI: now also C153.4.1, R153.4.1, TP153.4.TP; no longer C153.2.1, D152.C, R159.1, TP153.2.TP
- net GAIN1+: now also IC101.1A.RG@1, R101.1.2, TP104.1.TP; no longer IC111A.RG@1, R111.2, TP116.TP
- net GAIN1-: now also IC101.1A.RG, R101.1.1, TP103.1.TP; no longer IC111A.RG, R111.1, TP115.TP
- net GAIN2+: now also IC101.2A.RG@1, R101.2.2, TP104.2.TP; no longer IC121A.RG@1, R121.2, TP126.TP
- net GAIN2-: now also IC101.2A.RG, R101.2.1, TP103.2.TP; no longer IC121A.RG, R121.1, TP125.TP
- net GAIN3+: now also IC101.3A.RG@1, R101.3.2, TP104.3.TP; no longer IC101.1A.RG@1, R101.1.2, TP104.1.TP
- net GAIN3-: now also IC101.3A.RG, R101.3.1, TP103.3.TP; no longer IC101.1A.RG, R101.1.1, TP103.1.TP
- net GAIN4+: now also IC101.4A.RG@1, R101.4.2, TP104.4.TP; no longer IC101.2A.RG@1, R101.2.2, TP104.2.TP
- net GAIN4-: now also IC101.4A.RG, R101.4.1, TP103.4.TP; no longer IC101.2A.RG, R101.2.1, TP103.2.TP
- net GAIN_B0_DO: now also R159.1; no longer R92.1
- net GAIN_B1_DO: now also R157.1; no longer R91.1
- net IN1+: now also C105.1.2, IC101.1A.+IN, JP101.1.2, L102.1.1, TP102.1.TP; no longer C111.2, IC111A.+IN, JP111.2, L112.1, TP114.TP
- net IN1-: now also C105.1.1, IC101.1A.-IN, JP101.1.1, L101.1.1, TP101.1.TP; no longer C111.1, IC111A.-IN, JP111.1, L111.1, TP113.TP
- net IN2+: now also C105.2.2, IC101.2A.+IN, JP101.2.2, L102.2.1, TP102.2.TP; no longer C121.2, IC121A.+IN, JP121.2, L122.1, TP124.TP
- net IN2-: now also C105.2.1, IC101.2A.-IN, JP101.2.1, L101.2.1, TP101.2.TP; no longer C121.1, IC121A.-IN, JP121.1, L121.1, TP123.TP
- net IN3+: now also C105.3.2, IC101.3A.+IN, JP101.3.2, L102.3.1, TP102.3.TP; no longer C105.1.2, IC101.1A.+IN, JP101.1.2, L102.1.1, TP102.1.TP
- net IN3-: now also C105.3.1, IC101.3A.-IN, JP101.3.1, L101.3.1, TP101.3.TP; no longer C105.1.1, IC101.1A.-IN, JP101.1.1, L101.1.1, TP101.1.TP
- net IN4+: now also C105.4.2, IC101.4A.+IN, JP101.4.2, L102.4.1, TP102.4.TP; no longer C105.2.2, IC101.2A.+IN, JP101.2.2, L102.2.1, TP102.2.TP
- net IN4-: now also C105.4.1, IC101.4A.-IN, JP101.4.1, L101.4.1, TP101.4.TP; no longer C105.2.1, IC101.2A.-IN, JP101.2.1, L101.2.1, TP101.2.TP
- net SD_SPI_MISO_DI: now also U21.1.DO, U21.2.DO; no longer U1.DO
- net SD_SPI_MOSI_DO: now also IC4.DIN, U21.1.DI, U21.2.DI; no longer U1.DI
- net SD_SPI_SCK_DO: now also IC4.SCLK, U21.1.CLK, U21.2.CLK; no longer U1.CLK
- net SENSE1+: now also D51.1.C, L102.1.2, X101.1G1.1; no longer JP112.2, L112.2, TP112.TP, X111G1.1
- net SENSE1-: now also L101.1.2, X101.1G1.GND, X101.1G2.GND, X101.1G3.GND, X101.1G4.GND; no longer L111.2, TP111.TP, X111G1.GND, X111G2.GND, X111G3.GND, X111G4.GND
- net SENSE2+: now also D51.2.C, L102.2.2, X101.2G1.1; no longer JP122.2, L122.2, TP122.TP, X121G1.1
- net SENSE2-: now also L101.2.2, X101.2G1.GND, X101.2G2.GND, X101.2G3.GND, X101.2G4.GND; no longer L121.2, TP121.TP, X121G1.GND, X121G2.GND, X121G3.GND, X121G4.GND
- net SENSE3+: now also D51.3.C, L102.3.2, X101.3G1.1; no longer JP132.2, L102.1.2, TP132.TP, X101.1G1.1
- net SENSE3-: now also L101.3.2, X101.3G1.GND, X101.3G2.GND, X101.3G3.GND, X101.3G4.GND; no longer L101.1.2, TP131.TP, X101.1G1.GND, X101.1G2.GND, X101.1G3.GND, X101.1G4.GND
- net SENSE4+: now also D51.4.C, L102.4.2, X101.4G1.1; no longer JP142.2, L102.2.2, TP142.TP, X101.2G1.1
- net SENSE4-: now also L101.4.2, X101.4G1.GND, X101.4G2.GND, X101.4G3.GND, X101.4G4.GND; no longer L101.2.2, TP141.TP, X101.2G1.GND, X101.2G2.GND, X101.2G3.GND, X101.2G4.GND
- net TC1+: now also L301.1.2; no longer L301.2
- net TC1-: now also L302.1.2; no longer L302.2
- net TC2+: now also L301.2.2; no longer L303.2
- net TC2-: now also L302.2.2; no longer L304.2
- net TC3+: now also L301.3.2; no longer L305.2
- net TC3-: now also L302.3.2; no longer L306.2
- net TC4+: now also L301.4.2; no longer L307.2
- net TC4-: now also L302.4.2; no longer L308.2
- net TEMP_SPI_MISO_DI: now also IC301.1A.MISO, IC301.2A.MISO, IC301.3A.MISO, IC301.4A.MISO; no longer IC301A.MISO, IC302A.MISO, IC303A.MISO, IC304A.MISO
- net TEMP_SPI_SCK_DO: now also IC301.1A.SCK, IC301.2A.SCK, IC301.3A.SCK, IC301.4A.SCK; no longer IC301A.SCK, IC302A.SCK, IC303A.SCK, IC304A.SCK
- net TK1_N: now also C301.1.2, IC301.1A.T-, L302.1.1; no longer C301.2, IC301A.T-, L302.1
- net TK1_P: now also C301.1.1, IC301.1A.T+, L301.1.1; no longer C301.1, IC301A.T+, L301.1
- net TK2_N: now also C301.2.2, IC301.2A.T-, L302.2.1; no longer C302.2, IC302A.T-, L304.1
- net TK2_P: now also C301.2.1, IC301.2A.T+, L301.2.1; no longer C302.1, IC302A.T+, L303.1
- net TK3_N: now also C301.3.2, IC301.3A.T-, L302.3.1; no longer C303.2, IC303A.T-, L306.1
- net TK3_P: now also C301.3.1, IC301.3A.T+, L301.3.1; no longer C303.1, IC303A.T+, L305.1
- net TK4_N: now also C301.4.2, IC301.4A.T-, L302.4.1; no longer C304.2, IC304A.T-, L308.1
- net TK4_P: now also C301.4.1, IC301.4A.T+, L301.4.1; no longer C304.1, IC304A.T+, L307.1
- net VOFFS_RR: now also IC41B.-IN, R44.1.1, R45.1.2, TP46.1.TP; no longer IC31B.-IN, R35.1, R36.2, TP203.TP
- net VREF: now also C46.1, IC41A.+IN, IC42.C, R41.2, TP41.TP; no longer C35.1, IC31A.+IN, IC32.C, R31.1
- net VREF_2V5_BUFF: now also IC4.VREF, IC41A.-IN, IC41A.OUT, R34.A, R44.1.2, R44.2.2, R46.1.2, R46.2.2, TP42.TP; no longer IC31A.-IN, IC31A.OUT, R32.2, R35.2, TP201.TP
- net VREF_TRIM: now also R41.1.S, R42.1.1; no longer R33.S, R34.1
- net V_OFFS: now also C45.1.1, IC41B.+IN, R42.1.2, R43.1.2, TP45.1.TP; no longer C36.1, IC31B.+IN, JP31.1, R34.2, TP202.TP
- net V_OPREF1: now also C107.1.1, IC101.1A.REF, R103.1.2, TP107.1.TP; no longer C112.1, IC111A.REF, R112.2, TP117.TP
- net V_OPREF2: now also C107.2.1, IC101.2A.REF, R103.2.2, TP107.2.TP; no longer C122.1, IC121A.REF, R122.2, TP127.TP
- net V_OPREF3: now also C107.3.1, IC101.3A.REF, R103.3.2, TP107.3.TP; no longer C107.1.1, IC101.1A.REF, R103.1.2, TP107.1.TP
- net V_OPREF4: now also C107.4.1, IC101.4A.REF, R103.4.2, TP107.4.TP; no longer C107.2.1, IC101.2A.REF, R103.2.2, TP107.2.TP
Other:
- note added: "Numbering System: 10: Microcontroller 20: Flash Memory 30: DAC 40: Offset Voltage Generation 50: Current Sources 100: Diff-Amp CH1-4 150: Post-Amp Ch1-4 300: Thermocouples"
- note added: "Voltage reference"
- note removed: "Offset voltage reference"
- note removed: "Trim range: ~0.65mA - 7.1mA"
