File: 010_Hardware/010_uTTA_Eagle/uTTA_V2_Measure.sch (EAGLE design)
At the start: 303 parts, among them IC101.1 LT1167, IC101.2 LT1167, IC101.3 LT1167, IC101.4 LT1167, IC151.1 MCP602SN, IC151.3 MCP602SN, IC301 AD5664, IC302 LT1004CLP-2.5, IC303 TL074D, IC351.1 OPA2156ID, IC351.2 OPA2156ID, IC351.3 OPA2156ID, IC351.4 OPA2156ID, IC601.1 MAX6675ISA, IC601.2 MAX6675ISA, IC601.3 MAX6675ISA, IC601.4 MAX6675ISA, T151 BSS138PS, U11 NUCLEO_F103_BOT, U121.1 W25Q128JV, U121.2 W25Q128JV, X101.1 BU-SMA-GSPECIAL, X101.2 BU-SMA-GSPECIAL, X101.3 BU-SMA-GSPECIAL, X101.4 BU-SMA-GSPECIAL

Commit message: Optimization of Testpoints for Calibration
Parts:
- IC351.1, IC351.2, IC351.3, IC351.4: value OPA2156ID -> AD8672ARZ
- R326.1, R326.2: value 2k -> 4k99
- TP1, TP101.1, TP101.2, TP101.3, TP101.4, TP102.1, TP102.2, TP102.3, TP102.4, TP103.1, TP103.2, TP103.3, TP103.4, TP104.1, TP104.2, TP104.3, TP104.4, TP105.1, TP105.2, TP105.3, TP105.4, TP107.1, TP107.2, TP107.3, TP107.4, TP152.1, TP152.2, TP153, TP154, TP301, TP302, TP304, TP306, TP321.1, TP321.2, TP322.1, TP322.2, TP351.1, TP351.2, TP351.3, TP351.4, TP352.1, TP352.2, TP352.3, TP352.4, TP353.1, TP353.2, TP353.3, TP353.4, TP354.2, TP354.3, TP354.4, TP355.1, TP355.2, TP355.3, TP355.4, TP9354.1: value TP -> TPC90; device A_Testpoint:TP -> A_Testpoint:TPC90
- TP323.1, TP323.2: value TP -> TPO210H120; device A_Testpoint:TP -> A_Testpoint:TPO210H120
Connections:
- net V_OFF1 renamed V_OFF0
- net V_OFF2_4 renamed V_OFF1_3
Other:
- note added: "CH4 not supported by Software"
- note added: "Testpoint for Offset Voltage Calibration"
- note added: "V_OFF0 = ~-1.24V...2.5V Step Width = ~57.07µV"
- note added: "Variant without DAC"
- moved on the sheet: TP323.1, TP323.2
