File: 010_Hardware/010_uTTA_Eagle/uTTA_V2.1_Measure.sch (EAGLE design)
At the start: 286 parts, among them IC101.1 LT1167, IC101.2 LT1167, IC101.3 LT1167, IC101.4 LT1167, IC151.1 MCP602SN, IC151.3 MCP602SN, IC301 AD5664, IC302 LT1004CLP-2.5, IC303 TL074D, IC351.1 AD8672ARZ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

Commit message: update of OpAmp Selection
Other:
- note added: "For less offset voltage: Replace with TLV2387 or OPA2376"
Changed lines of the file:
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@@
 <text x="118.11" y="102.235" size="1.27" layer="98" ratio="14">tau = 330ns
 fc = 482.3kHz</text>
+<text x="30.48" y="148.59" size="1.27" layer="98">For less offset voltage:
+Replace with
+TLV2387 or OPA2376</text>
 </plain>
 <instances>
@@
 <wire x1="7.62" y1="17.78" x2="7.62" y2="63.5" width="0.1524" layer="98" style="shortdash"/>
 <text x="7.62" y="64.77" size="1.4224" layer="98">CH3 not supported by Software</text>
+<text x="30.48" y="151.13" size="1.27" layer="98">For less offset voltage:
+Replace with
+TLV2387 or OPA2376</text>
 </plain>
 <instances>
