File: 010_Hardware/010_uTTA_Eagle/uTTA_V2.1_Measure.brd (EAGLE design)
At the start: 100.4 x 79 mm, 287 parts, among them IC101.1 LT1167, IC101.2 LT1167, IC101.3 LT1167, IC101.4 LT1167, IC151.1 MCP602SN, IC151.3 MCP602SN, IC301 AD5664, IC302 LT1004CLP-2.5, IC303 TL074D, IC351.1 AD8672ARZ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

Commit message: Change of Offset Voltage decoupling resistors
Changed decoupling resistors from 10 Ohm to 0Ohm to reduce incluence on measurement results
Parts:
- R103.1, R103.2, R103.3, R103.4: value 10R -> 0R
- moved C107.3 188.8 mm to (-130.7, 27.1)
- moved C153.2 188.8 mm to (-161.5, 59.8)
- moved C153.3 188.8 mm to (-161.5, 62.4)
- moved C153.4 188.8 mm to (-161.5, 64.9)
- moved C3 188.8 mm to (-138.7, 24.8)
- moved C305 188.8 mm to (-143.4, 46.1)
- moved C321.1 188.8 mm to (-138.3, 52.8)
- moved C351.3 188.8 mm to (-123.9, 12.2)
- moved C352.1 188.8 mm to (-157.6, 14.2)
- moved C352.4 188.8 mm to (-109.5, 14.3)
- moved C602.2 188.8 mm to (-186.9, 19.3)
- moved D151 188.8 mm to (-154.5, 35.1)
- moved D152 188.8 mm to (-154.5, 36.9)
- moved IC302 188.8 mm to (-134.0, 42.2)
- moved IC303 188.8 mm to (-136.2, 51.2)
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Routing:
- net V_OFF0: track 52.1 -> 53.4 mm, vias 1 -> 2
Other:
- board text added: "!TEMP_SPI_CSN0_DO"
- board text added: "!TEMP_SPI_CSN1_DO"
- board text added: "!TEMP_SPI_CSN2_DO"
- board text added: "!TEMP_SPI_CSN3_DO"
- board text added: "CURR_MEAS_AI"
- board text added: "DBG_IO1"
- board text added: "DBG_IO2"
- board text added: "DBG_IO3"
- board text added: "DBG_IO4"
- board text added: "DIODE0_OUT_AI"
- board text added: "DIODE1_OUT_AI"
- board text added: "DIODE2_OUT_AI"
- board text added: "DIODE3_OUT_AI"
- board text added: "GAIN_B0_DO"
- board text added: "GAIN_B1_DO"
- board text added: "PSU_ENABLE_DO"
- board text added: "PWSTG_ENABLE_DO"
- board text added: "PWSTG_PWR_EN_DO"
- board text added: "PWSTG_UVLO_DI"
- board text added: "TEMP_SPI_MISO_DI"
- board text added: "TEMP_SPI_SCK_DO"

Commit message: Update of ADC filter RC-values
Changed ADC filter values to reduce effect of sampling droop
Parts:
- C153.1: value 1n/25V -> 10n/25V
- C153.2, C153.3, C153.4: value 2.2n/25V -> 10n/25V
- R153.1: value 330R -> 120
- R153.2, R153.3, R153.4: value 1k2 -> 120
Changed lines of the file:
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@@
 <attribute name="VALUE" x="-136.93775" y="43.561" size="1.27" layer="28" font="vector" rot="MR0" align="center"/>
 </element>
-<element name="R153.1" library="A_Resistor" package="R0603" value="330R" x="-161.51225" y="52.73675" smashed="yes" rot="MR180">
+<element name="R153.1" library="A_Resistor" package="R0603" value="120" x="-161.51225" y="52.73675" smashed="yes" rot="MR180">
 <attribute name="PACKAGE" value="R0603" x="-161.51225" y="52.73675" size="1.778" layer="28" rot="MR180" display="off"/>
 <attribute name="NAME" x="-161.51225" y="52.73675" size="0.4064" layer="38" font="vector" rot="MR180" align="center"/>
@@
 <attribute name="VALUE" x="-148.1455" y="18.415" size="1.27" layer="28" font="vector" rot="MR180" align="center"/>
 </element>
-<element name="R153.2" library="A_Resistor" package="R0603" value="1k2" x="-161.544" y="57.75325" smashed="yes" rot="MR180">
+<element name="R153.2" library="A_Resistor" package="R0603" value="120" x="-161.544" y="57.75325" smashed="yes" rot="MR180">
 <attribute name="PACKAGE" value="R0603" x="-209.4865" y="54.4195" size="1.778" layer="28" rot="MR180" display="off"/>
 <attribute name="NAME" x="-161.544" y="57.75325" size="0.4064" layer="38" font="vector" rot="MR180" align="center"/>
@@
 <attribute name="VALUE" x="-132.1435" y="18.2245" size="1.27" layer="28" font="vector" rot="MR180" align="center"/>
 </element>
-<element name="R153.3" library="A_Resistor" package="R0603" value="1k2" x="-157.95625" y="61.05525" smashed="yes" rot="MR180">
+<element name="R153.3" library="A_Resistor" package="R0603" value="120" x="-157.95625" y="61.05525" smashed="yes" rot="MR180">
 <attribute name="PACKAGE" value="R0603" x="-207.3275" y="44.3865" size="1.778" layer="28" rot="MR180" display="off"/>
 <attribute name="NAME" x="-157.95625" y="61.05525" size="0.4064" layer="38" font="vector" rot="MR180" align="center"/>
@@
 <variant name="Controller Adjust" populate="no"/>
 </element>
-<element name="R153.4" library="A_Resistor" package="R0603" value="1k2" x="-157.988" y="63.627" smashed="yes" rot="MR180">
+<element name="R153.4" library="A_Resistor" package="R0603" value="120" x="-157.988" y="63.627" smashed="yes" rot="MR180">
 <attribute name="PACKAGE" value="R0603" x="-223.0755" y="225.39325" size="1.778" layer="28" rot="MR180" display="off"/>
 <attribute name="NAME" x="-157.988" y="63.627" size="0.4064" layer="38" font="vector" rot="MR180" align="center"/>
@@
 <attribute name="VALUE" x="-122.047" y="47.46625" size="1.27" layer="27" font="vector" rot="R90" align="center"/>
 </element>
-<element name="C153.3" library="A_Kondensatoren" package="C0603" value="2.2n/25V" x="-161.544" y="62.357" smashed="yes" rot="MR180">
+<element name="C153.3" library="A_Kondensatoren" package="C0603" value="10n/25V" x="-161.544" y="62.357" smashed="yes" rot="MR180">
 <attribute name="PACKAGE" value="C0603" x="-161.544" y="62.357" size="1.778" layer="28" rot="MR180" display="off"/>
 <attribute name="NAME" x="-161.544" y="62.357" size="0.6096" layer="38" font="vector" rot="MR180" align="center"/>
@@
 <attribute name="NAME" x="-156.845" y="62.32525" size="1.27" layer="26" font="vector" rot="MR180" align="center"/>
 </element>
-<element name="C153.4" library="A_Kondensatoren" package="C0603" value="2.2n/25V" x="-161.544" y="64.897" smashed="yes" rot="MR180">
+<element name="C153.4" library="A_Kondensatoren" package="C0603" value="10n/25V" x="-161.544" y="64.897" smashed="yes" rot="MR180">
 <attribute name="PACKAGE" value="C0603" x="-161.544" y="64.897" size="1.778" layer="28" rot="MR180" display="off"/>
 <attribute name="NAME" x="-161.544" y="64.897" size="0.6096" layer="38" font="vector" rot="MR180" align="center"/>
@@
 <variant name="Controller Adjust" populate="no"/>
 </element>
-<element name="C153.2" library="A_Kondensatoren" package="C0603" value="2.2n/25V" x="-161.544" y="59.817" smashed="yes" rot="MR180">
+<element name="C153.2" library="A_Kondensatoren" package="C0603" value="10n/25V" x="-161.544" y="59.817" smashed="yes" rot="MR180">
 <attribute name="PACKAGE" value="C0603" x="-161.544" y="59.817" size="1.778" layer="28" rot="MR180" display="off"/>
 <attribute name="NAME" x="-161.544" y="59.817" size="0.6096" layer="38" font="vector" rot="MR180" align="center"/>
@@
 <attribute name="NAME" x="-156.7815" y="59.817" size="1.27" layer="26" font="vector" rot="MR180" align="center"/>
 </element>
-<element name="C153.1" library="A_Kondensatoren" package="C0603" value="1n/25V" x="-161.51225" y="54.76875" smashed="yes" rot="MR180">
+<element name="C153.1" library="A_Kondensatoren" package="C0603" value="10n/25V" x="-161.51225" y="54.76875" smashed="yes" rot="MR180">
 <attribute name="PACKAGE" value="C0603" x="-161.51225" y="54.76875" size="1.778" layer="28" rot="MR180" display="off"/>
 <attribute name="NAME" x="-161.51225" y="54.76875" size="0.6096" layer="38" font="vector" rot="MR180" align="center"/>
