File: 010_Hardware/010_uTTA_Eagle/uTTA_V1_Power.brd (EAGLE design)
At the start: 84 x 90.5 mm, 125 parts, among them IC1 MCP14E09, IC101 78L05SMD, IC102 7905ACM, IC103 LM393D, IC105 LT1167, IC2 SFH6156, IC3 SFH6156, IC4 SFH6156, J102 PIN23866A.68, J103 PIN23866A.68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

Commit message: Minor Cleanup of Design
Connections:
- net N$27 renamed VDD
- removed net E5V: U201.L_E5V
- net +5V: now also U201.L_E5V
Changed lines of the file:
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@@
 <contactref element="U201" pad="L_5V"/>
-</signal>
-<signal name="E5V">
-<contactref element="U201" pad="L_E5V"/>
 </signal>
 <signal name="AVDD">
@@
 <wire x1="14.12625" y1="9.205" x2="14.12875" y2="9.2075" width="0.6096" layer="16"/>
 <via x="14.12875" y="9.2075" extent="1-16" drill="0.3"/>
+<contactref element="U201" pad="L_E5V"/>
 </signal>
 <signal name="-5V">
@@
 <wire x1="49.68875" y1="11.5775" x2="49.7" y2="11.58875" width="0.6096" layer="1"/>
 </signal>
-<signal name="N$27">
-<contactref element="U201" pad="L_VDD"/>
-</signal>
 <signal name="N$6">
 <wire x1="4.15625" y1="53.53625" x2="1.3025" y2="53.53625" width="0.254" layer="1"/>
@@
 <wire x1="41.88975" y1="3.7465" x2="43.18" y2="2.45625" width="0.3048" layer="1"/>
 </signal>
+<signal name="VDD">
+<contactref element="U201" pad="L_VDD"/>
+</signal>
 </signals>

Commit message: Update on RC-filter values for current measurement
Parts:
- C1: value 1n/25V -> 22n/25V
- R117: value 330R -> 100R
Changed lines of the file:
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@@
 <clearance class="3" value="0.4"/>
+</class>
+<class number="9" name="GND" width="0.3" drill="0.3">
+<clearance class="0" value="0.2"/>
+<clearance class="1" value="0.2"/>
+<clearance class="2" value="0.2"/>
+<clearance class="3" value="0.3"/>
+<clearance class="4" value="0.2"/>
+<clearance class="5" value="0.25"/>
+<clearance class="6" value="0.25"/>
+<clearance class="7" value="0.4"/>
+<clearance class="8" value="0.4"/>
+<clearance class="9" value="0.2"/>
 </class>
 </classes>
@@
 <attribute name="PACKAGE" value="SO-8" x="47.9425" y="82.07375" size="1.778" layer="27" rot="R90" display="off"/>
 </element>
-<element name="R117" library="A_Resistor" package="R0603" value="330R" x="40.79875" y="82.70875" smashed="yes">
+<element name="R117" library="A_Resistor" package="R0603" value="100R" x="40.79875" y="82.70875" smashed="yes">
 <attribute name="NAME" x="34.44875" y="82.07375" size="1.27" layer="37"/>
 <attribute name="VALUE" x="40.16375" y="80.80375" size="1.27" layer="27"/>
@@
 <attribute name="VALUE" x="25.31625" y="83.67625" size="1.27" layer="27" rot="R180"/>
 </element>
-<element name="C1" library="A_Kondensatoren" package="C0603" value="1n/25V" x="37.30625" y="68.8975" smashed="yes">
+<element name="C1" library="A_Kondensatoren" package="C0603" value="22n/25V" x="37.30625" y="68.8975" smashed="yes">
 <attribute name="PACKAGE" value="C0603" x="37.30625" y="68.8975" size="1.778" layer="27" display="off"/>
 <attribute name="NAME" x="39.90975" y="68.3895" size="1.27" layer="37"/>
