File: 010_Hardware/010_uTTA_Eagle/uTTA_V1_Power.sch (EAGLE design)
At the start: 124 parts, among them IC1 MCP14E09, IC101 78L05SMD, IC102 7905ACM, IC103 LM393D, IC105 LT1167, IC2 SFH6156, IC3 SFH6156, IC4 SFH6156, J102 PIN23866A.68, J103 PIN23866A.68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

Commit message: Minor Cleanup of Design
Connections:
- removed net N$27: U201A.VDD
- net +5V: now also U201A.E5V
Changed lines of the file:
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@@
 <setting verticaltext="up"/>
 </settings>
-<grid distance="0.1" unitdist="inch" unit="inch" style="lines" multiple="1" display="no" altdistance="0.01" altunitdist="inch" altunit="inch"/>
+<grid distance="0.05" unitdist="inch" unit="inch" style="lines" multiple="1" display="no" altdistance="0.01" altunitdist="inch" altunit="inch"/>
 <layers>
 <layer number="1" name="Top" color="4" fill="1" visible="no" active="no"/>
@@
 <part name="G1" library="battery" deviceset="CR2032H" device=""/>
 <part name="AGND10" library="supply" deviceset="AGND_" device=""/>
+<part name="V10" library="A_Supply" deviceset="+8V" device="" value="+5V"/>
+<part name="AGND11" library="supply" deviceset="AGND_" device=""/>
 </parts>
 <sheets>
@@
 <instance part="U201" gate="B" x="170.18" y="130.81"/>
 <instance part="AGND4" gate="G$1" x="38.1" y="128.27"/>
-<instance part="V19" gate="G$1" x="102.87" y="142.24"/>
+<instance part="V19" gate="G$1" x="121.92" y="140.97"/>
 <instance part="AGND5" gate="G$1" x="101.6" y="128.27"/>
 <instance part="AGND24" gate="G$1" x="132.08" y="139.7"/>
@@
 </instance>
 <instance part="AGND10" gate="G$1" x="33.02" y="95.25"/>
+<instance part="V10" gate="G$1" x="121.92" y="151.13"/>
+<instance part="AGND11" gate="G$1" x="101.6" y="143.51"/>
 </instances>
 <busses>
@@
 </segment>
 <segment>
+<pinref part="U201" gate="A" pin="GND"/>
+<wire x1="96.52" y1="146.05" x2="101.6" y2="146.05" width="0.1524" layer="91"/>
+<pinref part="AGND11" gate="G$1" pin="AGND"/>
+</segment>
+<segment>
 <pinref part="U201" gate="A" pin="GND@3"/>
 <wire x1="96.52" y1="128.27" x2="99.06" y2="128.27" width="0.1524" layer="91"/>
@@
 <pinref part="U201" gate="A" pin="GND@1"/>
 <wire x1="96.52" y1="130.81" x2="99.06" y2="130.81" width="0.1524" layer="91"/>
-<pinref part="U201" gate="A" pin="GND"/>
-<wire x1="96.52" y1="146.05" x2="99.06" y2="146.05" width="0.1524" layer="91"/>
-<wire x1="99.06" y1="146.05" x2="99.06" y2="130.81" width="0.1524" layer="91"/>
 <junction x="99.06" y="130.81"/>
 </segment>
@@
 <pinref part="V19" gate="G$1" pin="+3V3"/>
 <pinref part="U201" gate="A" pin="3V3"/>
-<wire x1="96.52" y1="135.89" x2="102.87" y2="135.89" width="0.1524" layer="91"/>
-<wire x1="102.87" y1="135.89" x2="102.87" y2="139.7" width="0.1524" layer="91"/>
+<wire x1="96.52" y1="135.89" x2="121.92" y2="135.89" width="0.1524" layer="91"/>
+<wire x1="121.92" y1="135.89" x2="121.92" y2="138.43" width="0.1524" layer="91"/>
 </segment>
 </net>
@@
 <pinref part="U201" gate="A" pin="NC2"/>
 <wire x1="63.5" y1="143.51" x2="38.1" y2="143.51" width="0.1524" layer="91"/>
+</segment>
+<segment>
+<pinref part="V10" gate="G$1" pin="+8V"/>
+<wire x1="121.92" y1="151.13" x2="121.92" y2="148.59" width="0.1524" layer="91"/>
+<wire x1="96.52" y1="148.59" x2="121.92" y2="148.59" width="0.1524" layer="91"/>
+<pinref part="U201" gate="A" pin="E5V"/>
 </segment>
 </net>
@@
 </segment>
 </net>
-<net name="N$27" class="0">
-<segment>
-<pinref part="U201" gate="A" pin="VDD"/>
-<wire x1="63.5" y1="148.59" x2="55.88" y2="148.59" width="0.1524" layer="91"/>
-</segment>
-</net>

Commit message: Update on RC-filter values for current measurement
Parts:
- C1: value 1n/25V -> 22n/25V
- R117: value 330R -> 100R
Other:
- note added: "AV = 50V/V 30A -> 1.5V ~12.2mA/digit tau = 2.2µs fc = 72.343kHz"
Changed lines of the file:
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@@
 <setting verticaltext="up"/>
 </settings>
-<grid distance="0.05" unitdist="inch" unit="inch" style="lines" multiple="1" display="no" altdistance="0.01" altunitdist="inch" altunit="inch"/>
+<grid distance="0.1" unitdist="inch" unit="inch" style="lines" multiple="1" display="no" altdistance="0.01" altunitdist="inch" altunit="inch"/>
 <layers>
 <layer number="1" name="Top" color="4" fill="1" visible="no" active="no"/>
@@
 <layer number="101" name="TC_K" color="13" fill="1" visible="yes" active="yes"/>
 <layer number="102" name="bot_pads" color="7" fill="1" visible="yes" active="yes"/>
+<layer number="103" name="fp3" color="7" fill="1" visible="no" active="yes"/>
 <layer number="104" name="S_DOKU" color="7" fill="1" visible="yes" active="yes"/>
 <layer number="105" name="Beschreib" color="9" fill="1" visible="no" active="no"/>
@@
 <layer number="117" name="GROUND" color="16" fill="1" visible="yes" active="yes"/>
 <layer number="118" name="Rect_Pads" color="7" fill="1" visible="no" active="no"/>
+<layer number="121" name="_tsilk" color="7" fill="1" visible="no" active="yes"/>
+<layer number="122" name="_bsilk" color="7" fill="1" visible="no" active="yes"/>
 <layer number="123" name="tTestmark" color="7" fill="1" visible="no" active="no"/>
 <layer number="124" name="bTestmark" color="7" fill="1" visible="no" active="no"/>
@@
 <layer number="131" name="tAdjust" color="7" fill="1" visible="no" active="no"/>
 <layer number="132" name="bAdjust" color="7" fill="1" visible="no" active="no"/>
+<layer number="144" name="Drill_legend" color="7" fill="1" visible="no" active="yes"/>
 <layer number="150" name="Notes" color="7" fill="1" visible="yes" active="yes"/>
+<layer number="151" name="HeatSink" color="7" fill="1" visible="no" active="yes"/>
 <layer number="152" name="_bDocu" color="7" fill="1" visible="no" active="no"/>
 <layer number="153" name="FabDoc1" color="6" fill="1" visible="no" active="no"/>
@@
 <layer number="201" name="201bmp" color="2" fill="1" visible="no" active="no"/>
 <layer number="202" name="202bmp" color="3" fill="1" visible="no" active="no"/>
+<layer number="203" name="203bmp" color="4" fill="10" visible="no" active="yes"/>
+<layer number="204" name="204bmp" color="5" fill="10" visible="no" active="yes"/>
+<layer number="205" name="205bmp" color="6" fill="10" visible="no" active="yes"/>
+<layer number="206" name="206bmp" color="7" fill="10" visible="no" active="yes"/>
+<layer number="207" name="207bmp" color="8" fill="10" visible="no" active="yes"/>
+<layer number="208" name="208bmp" color="9" fill="10" visible="no" active="yes"/>
+<layer number="209" name="209bmp" color="7" fill="1" visible="no" active="yes"/>
+<layer number="210" name="210bmp" color="7" fill="1" visible="no" active="yes"/>
+<layer number="211" name="211bmp" color="7" fill="1" visible="no" active="yes"/>
+<layer number="212" name="212bmp" color="7" fill="1" visible="no" active="yes"/>
+<layer number="213" name="213bmp" color="7" fill="1" visible="no" active="yes"/>
+<layer number="214" name="214bmp" color="7" fill="1" visible="no" active="yes"/>
+<layer number="215" name="215bmp" color="7" fill="1" visible="no" active="yes"/>
+<layer number="216" name="216bmp" color="7" fill="1" visible="no" active="yes"/>
 <layer number="217" name="217bmp" color="18" fill="1" visible="no" active="no"/>
 <layer number="218" name="218bmp" color="19" fill="1" visible="no" active="no"/>
@@
 <clearance class="3" value="0.4"/>
 </class>
+<class number="9" name="GND" width="0.3" drill="0.3">
+<clearance class="0" value="0.2"/>
+<clearance class="1" value="0.2"/>
+<clearance class="2" value="0.2"/>
+<clearance class="3" value="0.3"/>
+<clearance class="4" value="0.2"/>
+<clearance class="5" value="0.25"/>
+<clearance class="6" value="0.25"/>
+<clearance class="7" value="0.4"/>
+<clearance class="8" value="0.4"/>
+<clearance class="9" value="0.2"/>
+</class>
 </classes>
 <parts>
@@
 <part name="AGND1" library="supply" deviceset="AGND_" device=""/>
 <part name="IC105" library="A_Linear_Technology" deviceset="LT1167" device=""/>
-<part name="R117" library="A_Resistor" deviceset="R-EU_" device="R0603" value="330R"/>
+<part name="R117" library="A_Resistor" deviceset="R-EU_" device="R0603" value="100R"/>
 <part name="AGND9" library="supply" deviceset="AGND_" device=""/>
 <part name="X101" library="A_Steckverbinder" deviceset="AST_03" device="_3,5MM_45°" value="AST_03_3,5MM"/>
@@
 <part name="9VS4" library="supply" deviceset="+12V" device="" value="+9VS"/>
 <part name="X1" library="A_Steckverbinder" deviceset="AST_02" device="_3,5MM_45°"/>
-<part name="C1" library="A_Kondensatoren" deviceset="C-EU" device="C0603" value="1n/25V"/>
+<part name="C1" library="A_Kondensatoren" deviceset="C-EU" device="C0603" value="22n/25V"/>
 <part name="AGND3" library="supply" deviceset="AGND_" device=""/>
 <part name="D1" library="A_Dioden" deviceset="DIODE-" device="SOD123" value="BAT46W"/>
@@
 <text x="116.205" y="85.725" size="1.27" layer="98">Replaceable with INA128</text>
 <text x="40.64" y="115.57" size="1.27" layer="98">UF=1.7V @ 16mA</text>
-<text x="99.695" y="58.42" size="1.4224" layer="98">AV = 50V/V
+<text x="97.155" y="53.34" size="1.4224" layer="98">AV = 50V/V
 30A -&gt; 1.5V
-~12.2mA/digit</text>
+~12.2mA/digit
+tau = 2.2µs
+fc = 72.343kHz</text>
 <wire x1="3.81" y1="44.45" x2="100.33" y2="44.45" width="0.4064" layer="98"/>
 <wire x1="100.33" y1="44.45" x2="100.33" y2="1.27" width="0.4064" layer="98"/>
