File: 010_Hardware/010_uTTA_Eagle/uTTA_V2.2_Power.brd (EAGLE design)
At the start: 84 x 90.5 mm, 125 parts, among them IC1 MCP14E09, IC101 78L05SMD, IC102 7905ACM, IC103 LM393D, IC105 LT1167, IC2 SFH6156, IC3 SFH6156, IC4 SFH6156, J102 PIN23866A.68, J103 PIN23866A.68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

Commit message: Update to uTTA Version 2.2
Full update of both PCBs to HW Version 2.2:
Removed spare FLASH Memory
Adjusted Position of LEDs and Buttons
Cleanup of layout
Parts:
- R126, R127: value 10R -> DNP
- R128: value 4m -> DNP
- moved C4 0.79 mm to (77.8, 64.3)
- moved C3 0.32 mm to (69.1, 58.6)
Other:
- board text added: "PGOOD"
- board text added: "µTTA V2.2"
- board text removed: "LO BATT"
- board text removed: "µTTA V1"

Commit message: changed resistor values
Changed Values of R101 and R102 to 0 Ohm
Changed value of R108 from 100 Ohm to 240 Ohm (to reduce optocoupler LED current)
Changed value of R110 from 220 Ohm to 470 Ohm (to reduce LED current)
Parts:
- R101, R102: value 10 -> 0
- R108: value 100R -> 240R
- R110: value 270R -> 470R
Other:
- board text added: ">VERSION"
- board text added: "µTTA"
- board text removed: "µTTA V2.2"
Changed lines of the file:
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@@
 <grid distance="6.25" unitdist="mil" unit="mm" style="lines" multiple="1" display="no" altdistance="0.025" altunitdist="inch" altunit="inch"/>
 <layers>
-<layer number="1" name="Top" color="4" fill="1" visible="no" active="yes"/>
+<layer number="1" name="Top" color="4" fill="1" visible="yes" active="yes"/>
 <layer number="2" name="Route2" color="22" fill="1" visible="no" active="yes"/>
 <layer number="15" name="Route15" color="18" fill="1" visible="no" active="yes"/>
-<layer number="16" name="Bottom" color="1" fill="1" visible="yes" active="yes"/>
+<layer number="16" name="Bottom" color="1" fill="1" visible="no" active="yes"/>
 <layer number="17" name="Pads" color="2" fill="1" visible="yes" active="yes"/>
 <layer number="18" name="Vias" color="2" fill="1" visible="yes" active="yes"/>
-<layer number="19" name="Unrouted" color="6" fill="1" visible="yes" active="yes"/>
+<layer number="19" name="Unrouted" color="6" fill="1" visible="no" active="yes"/>
 <layer number="20" name="Dimension" color="15" fill="1" visible="yes" active="yes"/>
-<layer number="21" name="tPlace" color="7" fill="1" visible="no" active="yes"/>
-<layer number="22" name="bPlace" color="7" fill="1" visible="yes" active="yes"/>
+<layer number="21" name="tPlace" color="7" fill="1" visible="yes" active="yes"/>
+<layer number="22" name="bPlace" color="7" fill="1" visible="no" active="yes"/>
 <layer number="23" name="tOrigins" color="15" fill="1" visible="no" active="yes"/>
-<layer number="24" name="bOrigins" color="15" fill="1" visible="yes" active="yes"/>
-<layer number="25" name="tNames" color="7" fill="1" visible="no" active="yes"/>
-<layer number="26" name="bNames" color="7" fill="1" visible="yes" active="yes"/>
+<layer number="24" name="bOrigins" color="15" fill="1" visible="no" active="yes"/>
+<layer number="25" name="tNames" color="7" fill="1" visible="yes" active="yes"/>
+<layer number="26" name="bNames" color="7" fill="1" visible="no" active="yes"/>
 <layer number="27" name="tValues" color="7" fill="1" visible="no" active="yes"/>
 <layer number="28" name="bValues" color="7" fill="1" visible="no" active="yes"/>
@@
 <layer number="36" name="bGlue" color="7" fill="5" visible="no" active="yes"/>
 <layer number="37" name="tTest" color="7" fill="1" visible="no" active="yes"/>
-<layer number="38" name="bTest" color="7" fill="1" visible="yes" active="yes"/>
+<layer number="38" name="bTest" color="7" fill="1" visible="no" active="yes"/>
 <layer number="39" name="tKeepout" color="4" fill="11" visible="no" active="yes"/>
 <layer number="40" name="bKeepout" color="1" fill="11" visible="no" active="yes"/>
@@
 <layer number="47" name="Measures" color="7" fill="1" visible="no" active="yes"/>
 <layer number="48" name="Document" color="7" fill="1" visible="yes" active="yes"/>
-<layer number="49" name="Reference" color="7" fill="1" visible="yes" active="yes"/>
-<layer number="50" name="dxf" color="7" fill="1" visible="yes" active="yes"/>
-<layer number="51" name="tDocu" color="7" fill="1" visible="no" active="yes"/>
-<layer number="52" name="bDocu" color="7" fill="1" visible="yes" active="yes"/>
+<layer number="49" name="Reference" color="7" fill="1" visible="no" active="yes"/>
+<layer number="50" name="dxf" color="7" fill="1" visible="no" active="yes"/>
+<layer number="51" name="tDocu" color="7" fill="1" visible="yes" active="yes"/>
+<layer number="52" name="bDocu" color="7" fill="1" visible="no" active="yes"/>
 <layer number="91" name="Nets" color="2" fill="1" visible="no" active="no"/>
 <layer number="92" name="Busses" color="1" fill="1" visible="no" active="no"/>
@@
 <layer number="112" name="tSilk" color="7" fill="1" visible="no" active="no"/>
 <layer number="113" name="ReferenceLS" color="7" fill="1" visible="no" active="no"/>
-<layer number="114" name="PLUS" color="28" fill="1" visible="no" active="yes"/>
-<layer number="115" name="MINUS" color="25" fill="1" visible="no" active="yes"/>
+<layer number="114" name="PLUS" color="28" fill="1" visible="no" active="no"/>
+<layer number="115" name="MINUS" color="25" fill="1" visible="no" active="no"/>
 <layer number="116" name="Patch_BOT" color="7" fill="1" visible="no" active="no"/>
-<layer number="117" name="GROUND" color="16" fill="1" visible="no" active="yes"/>
+<layer number="117" name="GROUND" color="16" fill="1" visible="no" active="no"/>
 <layer number="118" name="Rect_Pads" color="7" fill="1" visible="no" active="no"/>
 <layer number="121" name="_tsilk" color="7" fill="1" visible="no" active="no"/>
@@
 <circle x="59.69" y="86.51875" radius="0.22450625" width="0.4064" layer="25"/>
 <circle x="68.10375" y="86.51875" radius="0.22450625" width="0.4064" layer="25"/>
-<text x="45.70375" y="40.5275" size="2.5" layer="25" font="vector" ratio="18" rot="R90" align="center-left">µTTA V2.2</text>
+<text x="45.8625" y="38.305" size="2.5" layer="25" font="vector" ratio="18" rot="R90" align="center-left">µTTA</text>
 <wire x1="42.37" y1="37.51125" x2="43.9575" y2="37.51125" width="0.254" layer="25"/>
 <circle x="41.1" y="37.51125" radius="1.2" width="0.254" layer="21"/>
@@
 <text x="3.6325" y="57.04" size="1.778" layer="15" font="vector" ratio="20" rot="R90" align="bottom-center">3</text>
 <text x="3.6325" y="59.42875" size="1.778" layer="16" font="vector" ratio="15" rot="R90" align="bottom-center">4</text>
+<text x="45.8625" y="48.465" size="2.5" layer="25" font="vector" ratio="18" rot="R90" align="center-left">&gt;VERSION</text>
 </plain>
 <attributes>
-<attribute name="VERSION" value="2.2"/>
+<attribute name="VERSION" value="2.5.3"/>
 </attributes>
 <variantdefs>
@@
 <attribute name="PACKAGE" value="R0603" x="81.5975" y="81.43875" size="1.778" layer="27" rot="R270" display="off"/>
 </element>
-<element name="R101" library="A_Resistor" package="R0805" value="10" x="14.12875" y="70.485" smashed="yes" rot="MR270">
+<element name="R101" library="A_Resistor" package="R0805" value="0" x="14.12875" y="70.485" smashed="yes" rot="MR270">
 <attribute name="NAME" x="13.0175" y="72.54875" size="1.27" layer="38" rot="MR270"/>
 <attribute name="VALUE" x="16.66875" y="71.12" size="1.27" layer="28" rot="MR270"/>
 <attribute name="PACKAGE" value="R0805" x="14.12875" y="70.485" size="1.778" layer="28" rot="MR270" display="off"/>
 </element>
-<element name="R102" library="A_Resistor" package="R0805" value="10" x="11.90625" y="70.485" smashed="yes" rot="MR270">
+<element name="R102" library="A_Resistor" package="R0805" value="0" x="11.90625" y="70.485" smashed="yes" rot="MR270">
 <attribute name="NAME" x="13.0175" y="68.42125" size="1.27" layer="38" rot="MR90"/>
 <attribute name="VALUE" x="14.44625" y="71.12" size="1.27" layer="28" rot="MR270"/>
@@
 <attribute name="PACKAGE" value="R0603" x="31.59125" y="22.225" size="1.778" layer="27" rot="R90" display="off"/>
 </element>
-<element name="R108" library="A_Resistor" package="R0603" value="100R" x="35.71875" y="26.51125" smashed="yes">
+<element name="R108" library="A_Resistor" package="R0603" value="240R" x="35.71875" y="26.51125" smashed="yes">
 <attribute name="NAME" x="37.62375" y="26.035" size="1.27" layer="37"/>
 <attribute name="VALUE" x="35.08375" y="24.60625" size="1.27" layer="27"/>
@@
 <attribute name="PACKAGE" value="SOT-23" x="25.7175" y="46.0375" size="1.778" layer="27" display="off"/>
 </element>
-<element name="R110" library="A_Resistor" package="R0603" value="270R" x="22.5425" y="46.355" smashed="yes" rot="R90">
+<element name="R110" library="A_Resistor" package="R0603" value="470R" x="22.5425" y="46.355" smashed="yes" rot="R90">
 <attribute name="NAME" x="21.59" y="44.45" size="1.27" layer="37" rot="R270"/>
 <attribute name="VALUE" x="24.4475" y="45.72" size="1.27" layer="27" rot="R90"/>
